Commit message: Implemented taxi drone, removed edges from 3d models and all beacons properly configured

File: src/BetaBot/beta_bot_description/urdf/main.xacro (robot description, xacro)
@@ -11,12 +11,12 @@
             </inertial>
             <visual>
-                <origin xyz="-0.35 -0.775 -0.6" rpy="0.0 0.0 0.0"/>
+                <origin xyz="0 0 0" rpy="0.0 0.0 0.0"/>
                 <geometry>
-                    <mesh filename="package://beta_bot_description/meshes/model.dae" scale="0.05 0.05 0.05"/>
+                    <mesh filename="package://beta_bot_description/meshes/taxi.dae" scale="0.5 0.5 0.5"/>
                 </geometry>
             </visual>
             <collision>
                 <geometry>
-                    <box size="2.25 2.25 1.5"/>
+                    <box size="4 4 3"/>
                 </geometry>
             </collision>

Commit message: SeLe/F: Collision model updated to mesh

File: src/BetaBot/beta_bot_description/urdf/main.xacro (robot description, xacro)
@@ -17,6 +17,7 @@
             </visual>
             <collision>
+                <origin xyz="0 0 0" rpy="0.0 0.0 0.0"/>
                 <geometry>
-                    <box size="4 4 3"/>
+                    <mesh filename="package://beta_bot_description/meshes/taxi.dae" scale="0.5 0.5 0.5"/>
                 </geometry>
             </collision>

Commit message: Added localization based on ROS package robot-localization #WIP

File: src/BetaBot/beta_bot_description/urdf/main.xacro (robot description, xacro)
@@ -19,4 +19,5 @@
                 <origin xyz="0 0 0" rpy="0.0 0.0 0.0"/>
                 <geometry>
+                    <!-- <box size="4 4 3"/> -->
                     <mesh filename="package://beta_bot_description/meshes/taxi.dae" scale="0.5 0.5 0.5"/>
                 </geometry>

Commit message: #F022: Ajustar parámetros físicos para evitar contactos extraños con suelo

File: src/BetaBot/beta_bot_description/urdf/main.xacro (robot description, xacro)
@@ -13,15 +13,39 @@
                 <origin xyz="0 0 0" rpy="0.0 0.0 0.0"/>
                 <geometry>
+                    <!-- <box size="4 4 3"/> -->
                     <mesh filename="package://beta_bot_description/meshes/taxi.dae" scale="0.5 0.5 0.5"/>
                 </geometry>
             </visual>
             <collision>
-                <origin xyz="0 0 0" rpy="0.0 0.0 0.0"/>
+                <origin xyz="0 0 -0.1" rpy="0.0 0.0 0.0"/>
                 <geometry>
                     <!-- <box size="4 4 3"/> -->
-                    <mesh filename="package://beta_bot_description/meshes/taxi.dae" scale="0.5 0.5 0.5"/>
+                    <mesh filename="package://beta_bot_description/meshes/collision.dae" scale="1 1 1"/>
                 </geometry>
             </collision>
         </link>
+        <gazebo reference="body">
+            <collision>
+                <surface>
+                    <friction>
+                        <ode>
+                            <mu>1000</mu>
+                            <mu2>1000</mu2>
+                        </ode>
+                    </friction>
+                    <bounce>
+                        <restitution_coefficient>1</restitution_coefficient>
+                        <threshold>0</threshold>
+                    </bounce>
+                    <contact>
+                        <ode>
+                            <kp>1000</kp>
+                            <kd>0</kd>
+                            <max_vel>1</max_vel>
+                        </ode>
+                    </contact>
+                </surface>
+            </collision>
+        </gazebo>
     </xacro:macro>
     <!-- LINKS AND JOINTS DESCRIPTION -->
