Commit message: Added localization based on ROS package robot-localization #WIP

File: src/BetaBot/beta_bot_description/urdf/include/quadrotor_sensors.gazebo.xacro (robot description, xacro)
@@ -2,4 +2,9 @@
 <robot xmlns:xacro="http://www.ros.org/wiki/xacro">
   <!-- Quadrotor Sensor Plugins -->
+   <!-- Forward facing camera -->
+    <xacro:include filename="$(find beta_bot_description)/urdf/include/generic_camera.urdf.xacro" />
+    <xacro:generic_camera name="front_cam" parent="base_link" ros_topic="camera/image" cam_info_topic="camera/camera_info" update_rate="30" res_x="640" res_y="480" image_format="R8G8B8" hfov="90">
+      <origin xyz="1.50 -0.0 -0.25" rpy="0 0 0"/>
+    </xacro:generic_camera>
   <xacro:macro name="quadrotor_sensors">
         <gazebo>
@@ -9,6 +14,6 @@
             <frameId>$(arg base_link_frame)</frameId>
             <topicName>raw_imu</topicName>
-            <rpyOffset>0 0 0</rpyOffset> <!-- deprecated -->
-            <gaussianNoise>0</gaussianNoise>  <!-- deprecated -->
+            <rpyOffset>0 0 0</rpyOffset>
+            <gaussianNoise>0</gaussianNoise>
             <accelDrift>0.5 0.5 0.5</accelDrift>
             <accelGaussianNoise>0.35 0.35 0.3</accelGaussianNoise>
@@ -23,5 +28,5 @@
             <altimeterTopicName>altimeter</altimeterTopicName>
             <offset>0</offset>
-            <drift>10.0</drift>
+            <drift>0.0</drift>
             <gaussianNoise>0.1</gaussianNoise>
           </plugin>
@@ -44,5 +49,5 @@
             <referenceLongitude>8.687077</referenceLongitude>
             <drift>5.0 5.0 5.0</drift>
-            <gaussianNoise>0.01 0.01 0.01</gaussianNoise>
+            <gaussianNoise>1.00 1.00 1.00</gaussianNoise>
             <velocityDrift>0 0 0</velocityDrift>
             <velocityGaussianNoise>0.05 0.05 0.05</velocityGaussianNoise>
@@ -56,4 +61,81 @@
           </plugin>
         </gazebo>
+        <!-- PLUGIN PROPIO -->
+        <gazebo reference="base_link"> <!-- Referencia al link donde se quiere conectar este sensor -->
+        <gravity>true</gravity>
+        <sensor name="imu_sensor" type="imu">
+          <always_on>true</always_on>
+          <update_rate>100</update_rate>
+          <visualize>true</visualize>
+          <topic>raw_imu3</topic>
+          <plugin filename="libgazebo_ros_imu_sensor.so" name="imu_plugin">
+            <topicName>raw_imu3</topicName>
+            <bodyName>base_link</bodyName>
+            <updateRateHZ>30.0</updateRateHZ>
+            <gaussianNoise>0.005</gaussianNoise>
+            <xyzOffset>0 0 0</xyzOffset>
+            <rpyOffset>0 0 0</rpyOffset>
+            <frameName>base_link</frameName>
+            <initialOrientationAsReference>false</initialOrientationAsReference>
+          </plugin>
+          <pose>0 0 0 0 0 0</pose>
+        </sensor>
+        </gazebo>
+        <gazebo reference="front_cam_link">
+          <sensor type="multicamera" name="stereo_camera">
+            <update_rate>30.0</update_rate>
+            <camera name="left">
+              <pose>0 0.035 0 0 0 0</pose>
+              <horizontal_fov>1.3962634</horizontal_fov>
+              <image>
+                <width>800</width>
+                <height>800</height>
+                <format>R8G8B8</format>
+              </image>
+              <clip>
+                <near>0.02</near>
+                <far>300</far>
+              </clip>
+              <noise>
+                <type>gaussian</type>
+                <mean>0.0</mean>
+                <stddev>0.007</stddev>
+              </noise>
+            </camera>
+            <camera name="right">
+              <pose>0 -0.035 0 0 0 0</pose>
+              <horizontal_fov>1.3962634</horizontal_fov>
+              <image>
+                <width>800</width>
+                <height>800</height>
+                <format>R8G8B8</format>
+              </image>
+              <clip>
+                <near>0.02</near>
+                <far>300</far>
+              </clip>
+              <noise>
+                <type>gaussian</type>
+                <mean>0.0</mean>
+                <stddev>0.007</stddev>
+              </noise>
+            </camera>
+            <plugin name="stereo_camera_controller" filename="libgazebo_ros_multicamera.so">
+              <alwaysOn>true</alwaysOn>
+              <updateRate>0.0</updateRate>
+              <cameraName>multisense_sl/camera</cameraName>
+              <imageTopicName>image_raw</imageTopicName>
+              <cameraInfoTopicName>camera_info</cameraInfoTopicName>
+              <frameName>stereo_camera_frame</frameName>
+              <!--<rightFrameName>right_camera_optical_frame</rightFrameName>-->
+              <hackBaseline>0.07</hackBaseline>
+              <distortionK1>0.0</distortionK1>
+              <distortionK2>0.0</distortionK2>
+              <distortionK3>0.0</distortionK3>
+              <distortionT1>0.0</distortionT1>
+              <distortionT2>0.0</distortionT2>
+            </plugin>
+          </sensor>
+        </gazebo>
   </xacro:macro>
 </robot>

File: src/BetaBot/beta_bot_description/urdf/main.xacro (robot description, xacro)
@@ -18,5 +18,6 @@
             <collision>
                 <geometry>
-                    <box size="4 4 3"/>
+                    <!-- <box size="4 4 3"/> -->
+                    <mesh filename="package://beta_bot_description/meshes/taxi.dae" scale="0.5 0.5 0.5"/>
                 </geometry>
             </collision>

Commit message: GPS coherence in code (not a functional change)

File: src/BetaBot/beta_bot_description/urdf/include/quadrotor_sensors.gazebo.xacro (robot description, xacro)
@@ -2,73 +2,73 @@
 <robot xmlns:xacro="http://www.ros.org/wiki/xacro">
   <!-- Quadrotor Sensor Plugins -->
-   <!-- Forward facing camera -->
-    <xacro:include filename="$(find beta_bot_description)/urdf/include/generic_camera.urdf.xacro" />
-    <xacro:generic_camera name="front_cam" parent="base_link" ros_topic="camera/image" cam_info_topic="camera/camera_info" update_rate="30" res_x="640" res_y="480" image_format="R8G8B8" hfov="90">
-      <origin xyz="1.50 -0.0 -0.25" rpy="0 0 0"/>
-    </xacro:generic_camera>
+  <!-- Forward facing camera -->
+  <xacro:include filename="$(find beta_bot_description)/urdf/include/generic_camera.urdf.xacro" />
+  <xacro:generic_camera name="front_cam" parent="base_link" ros_topic="camera/image" cam_info_topic="camera/camera_info" update_rate="30" res_x="640" res_y="480" image_format="R8G8B8" hfov="90">
+    <origin xyz="1.50 -0.0 -0.25" rpy="0 0 0"/>
+  </xacro:generic_camera>
   <xacro:macro name="quadrotor_sensors">
-        <gazebo>
-          <plugin name="quadrotor_baro_sim" filename="libhector_gazebo_ros_baro.so">
-            <updateRate>10.0</updateRate>
-            <bodyName>base_link</bodyName>
-            <frameId>$(arg base_link_frame)</frameId>
-            <topicName>pressure_height</topicName>
-            <altimeterTopicName>altimeter</altimeterTopicName>
-            <offset>0</offset>
-            <drift>0.0</drift>
-            <gaussianNoise>0.1</gaussianNoise>
-          </plugin>
-          <plugin name="quadrotor_magnetic_sim" filename="libhector_gazebo_ros_magnetic.so">
-            <updateRate>10.0</updateRate>
-            <bodyName>base_link</bodyName>
-            <frameId>$(arg base_link_frame)</frameId>
-            <topicName>magnetic</topicName>
-            <offset>0 0 0</offset>
-            <drift>0.0 0.0 0.0</drift>
-            <gaussianNoise>1.3e-2 1.3e-2 1.3e-2</gaussianNoise>
-          </plugin>
-          <plugin name="quadrotor_gps_sim" filename="libhector_gazebo_ros_gps.so">
-            <updateRate>4.0</updateRate>
-            <bodyName>base_link</bodyName>
-            <frameId>$(arg base_link_frame)</frameId>
-            <topicName>fix</topicName>
-            <velocityTopicName>fix_velocity</velocityTopicName>
-            <referenceLatitude>49.860246</referenceLatitude>
-            <referenceLongitude>8.687077</referenceLongitude>
-            <drift>5.0 5.0 5.0</drift>
-            <gaussianNoise>1.00 1.00 1.00</gaussianNoise>
-            <velocityDrift>0 0 0</velocityDrift>
-            <velocityGaussianNoise>0.05 0.05 0.05</velocityGaussianNoise>
-          </plugin>
-          <plugin name="quadrotor_groundtruth_sim" filename="libgazebo_ros_p3d.so">
-            <updateRate>100.0</updateRate>
-            <bodyName>base_link</bodyName>
-            <topicName>ground_truth/state</topicName>
-            <gaussianNoise>0.0</gaussianNoise>
-            <frameName>$(arg world_frame)</frameName>
-          </plugin>
-        </gazebo>
-        <!-- PLUGIN PROPIO -->
-        <gazebo reference="base_link">
-        <gravity>true</gravity>
-        <sensor name="imu_sensor" type="imu">
-          <always_on>true</always_on>
-          <update_rate>100</update_rate>
-          <visualize>true</visualize>
-          <topic>raw_imu3</topic>
-          <plugin filename="libgazebo_ros_imu_sensor.so" name="imu_plugin">
-            <topicName>raw_imu</topicName>
-            <bodyName>base_link</bodyName>
-            <updateRateHZ>30.0</updateRateHZ>
-            <gaussianNoise>0.005</gaussianNoise>
-            <xyzOffset>0 0 0</xyzOffset>
-            <rpyOffset>0 0 0</rpyOffset>
-            <frameName>base_link</frameName>
-            <initialOrientationAsReference>false</initialOrientationAsReference>
-          </plugin>
-          <pose>0 0 0 0 0 0</pose>
-        </sensor>
-        </gazebo>
-        <!-- IMU SERGI
+    <gazebo>
+      <plugin name="quadrotor_baro_sim" filename="libhector_gazebo_ros_baro.so">
+        <updateRate>10.0</updateRate>
+        <bodyName>base_link</bodyName>
+        <frameId>$(arg base_link_frame)</frameId>
+        <topicName>pressure_height</topicName>
+        <altimeterTopicName>altimeter</altimeterTopicName>
+        <offset>0</offset>
+        <drift>0.0</drift>
+        <gaussianNoise>0.1</gaussianNoise>
+      </plugin>
+      <plugin name="quadrotor_magnetic_sim" filename="libhector_gazebo_ros_magnetic.so">
+        <updateRate>10.0</updateRate>
+        <bodyName>base_link</bodyName>
+        <frameId>$(arg base_link_frame)</frameId>
+        <topicName>magnetic</topicName>
+        <offset>0 0 0</offset>
+        <drift>0.0 0.0 0.0</drift>
+        <gaussianNoise>1.3e-2 1.3e-2 1.3e-2</gaussianNoise>
+      </plugin>
+      <plugin name="quadrotor_gps_sim" filename="libhector_gazebo_ros_gps.so">
+        <updateRate>4.0</updateRate>
+        <bodyName>base_link</bodyName>
+        <frameId>$(arg base_link_frame)</frameId>
+        <topicName>/odometry/gps</topicName>
+        <velocityTopicName>fix_velocity</velocityTopicName>
+        <referenceLatitude>49.860246</referenceLatitude>
+        <referenceLongitude>8.687077</referenceLongitude>
+        <drift>5.0 5.0 5.0</drift>
+        <gaussianNoise>1.00 1.00 1.00</gaussianNoise>
+        <velocityDrift>0 0 0</velocityDrift>
+        <velocityGaussianNoise>0.05 0.05 0.05</velocityGaussianNoise>
+      </plugin>
+      <plugin name="quadrotor_groundtruth_sim" filename="libgazebo_ros_p3d.so">
+        <updateRate>100.0</updateRate>
+        <bodyName>base_link</bodyName>
+        <topicName>ground_truth/state</topicName>
+        <gaussianNoise>0.0</gaussianNoise>
+        <frameName>$(arg world_frame)</frameName>
+      </plugin>
+    </gazebo>
+    <!-- PLUGIN PROPIO -->
+    <gazebo reference="base_link">
+      <gravity>true</gravity>
+      <sensor name="imu_sensor" type="imu">
+        <always_on>true</always_on>
+        <update_rate>100</update_rate>
+        <visualize>true</visualize>
+        <topic>/raw_imu</topic>
+        <plugin filename="libgazebo_ros_imu_sensor.so" name="imu_plugin">
+          <topicName>/raw_imu</topicName>
+          <bodyName>base_link</bodyName>
+          <updateRateHZ>30.0</updateRateHZ>
+          <gaussianNoise>0.005</gaussianNoise>
+          <xyzOffset>0 0 0</xyzOffset>
+          <rpyOffset>0 0 0</rpyOffset>
+          <frameName>base_link</frameName>
+          <initialOrientationAsReference>false</initialOrientationAsReference>
+        </plugin>
+        <pose>0 0 0 0 0 0</pose>
+      </sensor>
+    </gazebo>
+    <!-- IMU SERGI
         <gazebo>
         <plugin name="imu_plugin" filename="libgazebo_ros_imu.so">
@@ -82,60 +82,60 @@
         </gazebo>
         -->
-        <gazebo reference="front_cam_link">
-          <sensor type="multicamera" name="stereo_camera">
-            <update_rate>30.0</update_rate>
-            <camera name="left">
-              <pose>0 0.035 0 0 0 0</pose>
-              <horizontal_fov>1.3962634</horizontal_fov>
-              <image>
-                <width>800</width>
-                <height>800</height>
-                <format>R8G8B8</format>
-              </image>
-              <clip>
-                <near>0.02</near>
-                <far>300</far>
-              </clip>
-              <noise>
-                <type>gaussian</type>
-                <mean>0.0</mean>
-                <stddev>0.007</stddev>
-              </noise>
-            </camera>
-            <camera name="right">
-              <pose>0 -0.035 0 0 0 0</pose>
-              <horizontal_fov>1.3962634</horizontal_fov>
-              <image>
-                <width>800</width>
-                <height>800</height>
-                <format>R8G8B8</format>
-              </image>
-              <clip>
-                <near>0.02</near>
-                <far>300</far>
-              </clip>
-              <noise>
-                <type>gaussian</type>
-                <mean>0.0</mean>
-                <stddev>0.007</stddev>
-              </noise>
-            </camera>
-            <plugin name="stereo_camera_controller" filename="libgazebo_ros_multicamera.so">
-              <alwaysOn>true</alwaysOn>
-              <updateRate>0.0</updateRate>
-              <cameraName>multisense_sl/camera</cameraName>
-              <imageTopicName>image_raw</imageTopicName>
-              <cameraInfoTopicName>camera_info</cameraInfoTopicName>
-              <frameName>stereo_camera_frame</frameName>
-              <!--<rightFrameName>right_camera_optical_frame</rightFrameName>-->
-              <hackBaseline>0.07</hackBaseline>
-              <distortionK1>0.0</distortionK1>
-              <distortionK2>0.0</distortionK2>
-              <distortionK3>0.0</distortionK3>
-              <distortionT1>0.0</distortionT1>
-              <distortionT2>0.0</distortionT2>
-            </plugin>
-          </sensor>
-        </gazebo>
+    <gazebo reference="front_cam_link">
+      <sensor type="multicamera" name="stereo_camera">
+        <update_rate>30.0</update_rate>
+        <camera name="left">
+          <pose>0 0.035 0 0 0 0</pose>
+          <horizontal_fov>1.3962634</horizontal_fov>
+          <image>
+            <width>800</width>
+            <height>800</height>
+            <format>R8G8B8</format>
+          </image>
+          <clip>
+            <near>0.02</near>
+            <far>300</far>
+          </clip>
+          <noise>
+            <type>gaussian</type>
+            <mean>0.0</mean>
+            <stddev>0.007</stddev>
+          </noise>
+        </camera>
+        <camera name="right">
+          <pose>0 -0.035 0 0 0 0</pose>
+          <horizontal_fov>1.3962634</horizontal_fov>
+          <image>
+            <width>800</width>
+            <height>800</height>
+            <format>R8G8B8</format>
+          </image>
+          <clip>
+            <near>0.02</near>
+            <far>300</far>
+          </clip>
+          <noise>
+            <type>gaussian</type>
+            <mean>0.0</mean>
+            <stddev>0.007</stddev>
+          </noise>
+        </camera>
+        <plugin name="stereo_camera_controller" filename="libgazebo_ros_multicamera.so">
+          <alwaysOn>true</alwaysOn>
+          <updateRate>0.0</updateRate>
+          <cameraName>multisense_sl/camera</cameraName>
+          <imageTopicName>image_raw</imageTopicName>
+          <cameraInfoTopicName>camera_info</cameraInfoTopicName>
+          <frameName>stereo_camera_frame</frameName>
+          <!--<rightFrameName>right_camera_optical_frame</rightFrameName>-->
+          <hackBaseline>0.07</hackBaseline>
+          <distortionK1>0.0</distortionK1>
+          <distortionK2>0.0</distortionK2>
+          <distortionK3>0.0</distortionK3>
+          <distortionT1>0.0</distortionT1>
+          <distortionT2>0.0</distortionT2>
+        </plugin>
+      </sensor>
+    </gazebo>
   </xacro:macro>
 </robot>
