Commit message: feat: 3d model camera added (intelsense stereo)

File: src/BetaBot/beta_bot_description/urdf/include/generic_camera.urdf.xacro (robot description, xacro)
@@ -9,24 +9,21 @@
     </joint>
     <link name="${name}_link">
-<!--      <inertial>
-        <mass value="0.001" />
+      <inertial>
+        <mass value="0.01" />
         <origin xyz="0 0 0" rpy="0 0 0" />
-        <inertia ixx="0.0001" ixy="0" ixz="0" iyy="0.0001" iyz="0" izz="0.0001" />
+        <inertia ixx="0.01" ixy="0" ixz="0" iyy="0.01" iyz="0" izz="0.01" />
       </inertial>
       <visual>
-        <origin xyz="0 0 0" rpy="0 0 0" />
+        <origin xyz="0 -0.25 0" rpy="0 0 ${pi/2}" />
         <geometry>
-          <box size="0.01 0.01 0.01" />
+          <mesh filename="package://beta_bot_description/meshes/camera.dae" scale="5 5 5"/>
         </geometry>
-        <material name="Blue">
-          <color rgba="0.0 0.0 0.8 1"/>
-        </material>
       </visual>
       <collision>
-        <origin xyz="0 0 0" rpy="0 0 0" />
+        <origin xyz="-0.1 -0.05 0.05" rpy="0 0 0" />
         <geometry>
-          <box size="0.01 0.01 0.01" />
+          <box size="0.1 0.5 0.1" />
         </geometry>
-      </collision>-->
+      </collision>
     </link>
     <joint name="${name}_optical_joint" type="fixed">

File: src/BetaBot/beta_bot_description/urdf/include/quadrotor_sensors.gazebo.xacro (robot description, xacro)
@@ -5,5 +5,5 @@
   <xacro:include filename="$(find beta_bot_description)/urdf/include/generic_camera.urdf.xacro" />
   <xacro:generic_camera name="front_cam" parent="base_link" ros_topic="camera/image" cam_info_topic="camera/camera_info" update_rate="30" res_x="640" res_y="480" image_format="R8G8B8" hfov="90">
-    <origin xyz="1.50 -0.0 -0.25" rpy="0 0 0"/>
+    <origin xyz="1.45 -0.0 -0.7" rpy="0 0 0"/>
   </xacro:generic_camera>
   <xacro:macro name="quadrotor_sensors">
